Commit message: Mega_update-coming-up!

File: 3D_PARTS/SpotMicro urdf/Assembly_For_Simulation_description - Copy (2)/urdf/Assembly_For_Simulation.urdf (robot description, URDF)
Before this commit: robot Assembly_For_Simulation, 13 links, 12 joints
Links:
- removed link LF_FOOT_1
- removed link LH_FOOT_1
- removed link RF_FOOT_1
- removed link RH_FOOT_1
- added link Back_left_forearm_1, mass 0.49369135494533783; collision mesh filename=package://Assembly_For_Simulation_description/meshes/Back_l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 scale=0.001 0.001 0.001; visual mesh filename=package://Assembly_For_Simulation_description/meshes/Back_l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 scale=0.001 0.001 0.001
- added link Back_right_forearm_1, mass 0.4997350884581435; collision mesh filename=package://Assembly_For_Simulation_description/meshes/Back_r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 scale=0.001 0.001 0.001; visual mesh filename=package://Assembly_For_Simulation_description/meshes/Back_r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 scale=0.001 0.001 0.001
- added link Front_left_forearm_1, mass 0.4907857835923385; collision mesh filename=package://Assembly_For_Simulation_description/meshes/Front_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 scale=0.001 0.001 0.001; visual mesh filename=package://Assembly_For_Simulation_description/meshes/Front_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 scale=0.001 0.001 0.001
- added link Front_right_forearm_1, mass 0.49985914540184717; collision mesh filename=package://Assembly_For_Simulation_description/meshes/Front_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 scale=0.001 0.001 0.001; visual mesh filename=package://Assembly_For_Simulation_description/meshes/Front_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 scale=0.001 0.001 0.001
Joints:
- joint BL_calf_joint: child LH_FOOT_1 -> Back_left_forearm_1
- joint BR_calf_joint: child RH_FOOT_1 -> Back_right_forearm_1
- joint FL_calf_joint: child LF_FOOT_1 -> Front_left_forearm_1
- joint FR_calf_joint: child RF_FOOT_1 -> Front_right_forearm_1

File: 3D_PARTS/SpotMicro urdf/Assembly_For_Simulation_description - Copy/urdf/Assembly_For_Simulation.xacro (robot description, xacro)
@@ -24,5 +24,5 @@
   </collision>
 </link>
-<link name="LH_FOOT_1">
+<link name="Back_left_forearm_1">
   <inertial>
     <origin xyz="-0.02387677244019979 0.02681764636693125 -0.014730802536600973" rpy="0 0 0"/>
@@ -33,5 +33,5 @@
     <origin xyz="-0.074761 -0.011235 -0.317307" rpy="0 0 0"/>
     <geometry>
-      <mesh filename="package://Assembly_For_Simulation_description/meshes/LH_FOOT_1.stl" scale="0.001 0.001 0.001"/>
+      <mesh filename="package://Assembly_For_Simulation_description/meshes/Back_left_forearm_1.stl" scale="0.001 0.001 0.001"/>
     </geometry>
     <material name="silver"/>
@@ -40,9 +40,9 @@
     <origin xyz="-0.074761 -0.011235 -0.317307" rpy="0 0 0"/>
     <geometry>
-      <mesh filename="package://Assembly_For_Simulation_description/meshes/LH_FOOT_1.stl" scale="0.001 0.001 0.001"/>
-    </geometry>
-  </collision>
-</link>
-<link name="RH_FOOT_1">
+      <mesh filename="package://Assembly_For_Simulation_description/meshes/Back_left_forearm_1.stl" scale="0.001 0.001 0.001"/>
+    </geometry>
+  </collision>
+</link>
+<link name="Back_right_forearm_1">
   <inertial>
     <origin xyz="0.027613181105729107 0.027492504385563943 -0.014145746962176853" rpy="0 0 0"/>
@@ -53,5 +53,5 @@
     <origin xyz="-0.220832 -0.007695 -0.315254" rpy="0 0 0"/>
     <geometry>
-      <mesh filename="package://Assembly_For_Simulation_description/meshes/RH_FOOT_1.stl" scale="0.001 0.001 0.001"/>
+      <mesh filename="package://Assembly_For_Simulation_description/meshes/Back_right_forearm_1.stl" scale="0.001 0.001 0.001"/>
     </geometry>
     <material name="silver"/>
@@ -60,9 +60,9 @@
     <origin xyz="-0.220832 -0.007695 -0.315254" rpy="0 0 0"/>
     <geometry>
-      <mesh filename="package://Assembly_For_Simulation_description/meshes/RH_FOOT_1.stl" scale="0.001 0.001 0.001"/>
-    </geometry>
-  </collision>
-</link>
-<link name="RF_FOOT_1">
+      <mesh filename="package://Assembly_For_Simulation_description/meshes/Back_right_forearm_1.stl" scale="0.001 0.001 0.001"/>
+    </geometry>
+  </collision>
+</link>
+<link name="Front_right_forearm_1">
   <inertial>
     <origin xyz="0.028280901609207154 0.03063734624089054 -0.014033926018012455" rpy="0 0 0"/>
@@ -73,5 +73,5 @@
     <origin xyz="-0.219953 -0.188311 -0.315701" rpy="0 0 0"/>
     <geometry>
-      <mesh filename="package://Assembly_For_Simulation_description/meshes/RF_FOOT_1.stl" scale="0.001 0.001 0.001"/>
+      <mesh filename="package://Assembly_For_Simulation_description/meshes/Front_right_forearm_1.stl" scale="0.001 0.001 0.001"/>
     </geometry>
     <material name="silver"/>
@@ -80,9 +80,9 @@
     <origin xyz="-0.219953 -0.188311 -0.315701" rpy="0 0 0"/>
     <geometry>
-      <mesh filename="package://Assembly_For_Simulation_description/meshes/RF_FOOT_1.stl" scale="0.001 0.001 0.001"/>
-    </geometry>
-  </collision>
-</link>
-<link name="LF_FOOT_1">
+      <mesh filename="package://Assembly_For_Simulation_description/meshes/Front_right_forearm_1.stl" scale="0.001 0.001 0.001"/>
+    </geometry>
+  </collision>
+</link>
+<link name="Front_left_forearm_1">
   <inertial>
     <origin xyz="-0.027057224103647512 0.03285362638972403 -0.0179332893641046" rpy="0 0 0"/>
@@ -93,5 +93,5 @@
     <origin xyz="-0.0789 -0.186175 -0.321641" rpy="0 0 0"/>
     <geometry>
-      <mesh filename="package://Assembly_For_Simulation_description/meshes/LF_FOOT_1.stl" scale="0.001 0.001 0.001"/>
+      <mesh filename="package://Assembly_For_Simulation_description/meshes/Front_left_forearm_1.stl" scale="0.001 0.001 0.001"/>
     </geometry>
     <material name="silver"/>
@@ -100,5 +100,5 @@
     <origin xyz="-0.0789 -0.186175 -0.321641" rpy="0 0 0"/>
     <geometry>
-      <mesh filename="package://Assembly_For_Simulation_description/meshes/LF_FOOT_1.stl" scale="0.001 0.001 0.001"/>
+      <mesh filename="package://Assembly_For_Simulation_description/meshes/Front_left_forearm_1.stl" scale="0.001 0.001 0.001"/>
     </geometry>
   </collision>
@@ -264,33 +264,33 @@
   </collision>
 </link>
-<joint name="BL_calf_joint" type="revolute">
+<joint name="Revolute 24" type="revolute">
   <origin xyz="-0.007078 -0.051761 -0.089937" rpy="0 0 0"/>
   <parent link="Back_left_upperarm_1"/>
-  <child link="LH_FOOT_1"/>
+  <child link="Back_left_forearm_1"/>
   <axis xyz="1.0 -0.000123 5e-05"/>
   <limit upper="0.785398" lower="-3.141593" effort="100" velocity="100"/>
 </joint>
-<joint name="BR_calf_joint" type="revolute">
+<joint name="Revolute 25" type="revolute">
   <origin xyz="0.002438 -0.05219 -0.092366" rpy="0 0 0"/>
   <parent link="Back_right_upperarm_1"/>
-  <child link="RH_FOOT_1"/>
+  <child link="Back_right_forearm_1"/>
   <axis xyz="-1.0 6.2e-05 -0.0"/>
   <limit upper="3.141593" lower="-0.785398" effort="100" velocity="100"/>
 </joint>
-<joint name="FR_calf_joint" type="revolute">
+<joint name="Revolute 26" type="revolute">
   <origin xyz="0.002862 -0.052497 -0.092075" rpy="0 0 0"/>
   <parent link="Front_right_upperarm_1"/>
-  <child link="RF_FOOT_1"/>
+  <child link="Front_right_forearm_1"/>
   <axis xyz="-1.0 6.2e-05 -0.0"/>
   <limit upper="3.141593" lower="-0.785398" effort="100" velocity="100"/>
 </joint>
-<joint name="FL_calf_joint" type="revolute">
+<joint name="Revolute 27" type="revolute">
   <origin xyz="-0.004287 -0.05781 -0.085759" rpy="0 0 0"/>
   <parent link="Front_left_upperarm_1"/>
-  <child link="LF_FOOT_1"/>
+  <child link="Front_left_forearm_1"/>
   <axis xyz="-1.0 0.000121 -5.2e-05"/>
   <limit upper="3.141593" lower="-0.785398" effort="100" velocity="100"/>
 </joint>
-<joint name="FL_thigh_joint" type="revolute">
+<joint name="Revolute 28" type="revolute">
   <origin xyz="-0.028042 -0.025573 -0.011445" rpy="0 0 0"/>
   <parent link="Front_left_shoulder_1"/>
@@ -299,5 +299,5 @@
   <limit upper="1.570796" lower="-2.96706" effort="100" velocity="100"/>
 </joint>
-<joint name="BL_thigh_joint" type="revolute">
+<joint name="Revolute 29" type="revolute">
   <origin xyz="-0.028727 -0.020217 -0.011601" rpy="0 0 0"/>
   <parent link="Back_left_shoulder_1"/>
@@ -306,5 +306,5 @@
   <limit upper="1.570796" lower="-2.96706" effort="100" velocity="100"/>
 </joint>
-<joint name="BR_thigh_joint" type="revolute">
+<joint name="Revolute 30" type="revolute">
   <origin xyz="0.028385 -0.023328 -0.011225" rpy="0 0 0"/>
   <parent link="Back_right_shoulder_1"/>
@@ -313,5 +313,5 @@
   <limit upper="1.570796" lower="-2.96706" effort="100" velocity="100"/>
 </joint>
-<joint name="FR_thigh_joint" type="revolute">
+<joint name="Revolute 31" type="revolute">
   <origin xyz="0.027745 -0.02875 -0.011069" rpy="0 0 0"/>
   <parent link="Front_right_shoulder_1"/>
@@ -320,5 +320,5 @@
   <limit upper="1.570796" lower="-2.96706" effort="100" velocity="100"/>
 </joint>
-<joint name="FL_hip_joint" type="revolute">
+<joint name="Revolute 32" type="revolute">
   <origin xyz="0.111229 0.269558 0.418845" rpy="0 0 0"/>
   <parent link="base_link"/>
@@ -327,5 +327,5 @@
   <limit upper="1.22173" lower="-1.047198" effort="100" velocity="100"/>
 </joint>
-<joint name="BL_hip_joint" type="revolute">
+<joint name="Revolute 33" type="revolute">
   <origin xyz="0.110566 0.083213 0.418845" rpy="0 0 0"/>
   <parent link="base_link"/>
@@ -334,5 +334,5 @@
   <limit upper="1.22173" lower="-1.047198" effort="100" velocity="100"/>
 </joint>
-<joint name="FR_hip_joint" type="revolute">
+<joint name="Revolute 34" type="revolute">
   <origin xyz="0.189346 0.269558 0.418845" rpy="0 0 0"/>
   <parent link="base_link"/>
@@ -341,5 +341,5 @@
   <limit upper="1.047198" lower="-1.22173" effort="100" velocity="100"/>
 </joint>
-<joint name="BR_hip_joint" type="revolute">
+<joint name="Revolute 35" type="revolute">
   <origin xyz="0.190009 0.083213 0.418845" rpy="0 0 0"/>
   <parent link="base_link"/>
